File: STMBreadboard.brd (EAGLE design)
At the start: 100 x 80 mm, 25 parts, among them IC1 REG1117, Y1 8MHz

Commit message: PCB002
Parts:
- added C4, C5: 47u, rcl:UD-6,3X7,7_NICHICON
- moved JP2 131.5 mm to (81.9, 31.8), turned to 180 degrees
- moved JP8 126.9 mm to (81.9, 49.5), turned to 180 degrees
- moved R6 123.7 mm to (81.9, 54.0), turned to 180 degrees
- moved LED4 113.9 mm to (84.5, 52.1), turned to 180 degrees
- moved JP4 106.8 mm to (72.4, 47.0), turned to 90 degrees
- moved JP1 93.9 mm to (55.9, 64.8)
- moved C3 86.9 mm to (69.8, 25.4), flipped to the bottom
- moved R1 85.2 mm to (69.8, 31.8)
- moved JP7 70.3 mm to (49.5, 34.9), turned to 270 degrees
- moved JP6 40.8 mm to (40.6, 47.0)
- moved S1 39.9 mm to (69.8, 25.4), turned to 270 degrees
- moved IC1 32.6 mm to (83.8, 44.5), flipped to the top, turned to 270 degrees
- moved C1 8.98 mm to (63.5, 22.9), flipped to the top
- moved C2 8.98 mm to (53.3, 22.9), flipped to the top
- moved JP5 3.81 mm to (58.4, 58.4), turned to 180 degrees
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Connections:
- net +3V3: now also C4.+
- net +5V: now also C5.+
- net GND: now also C4.-, C5.-
Routing:
- net GND: track 5.72 -> 185.6 mm
- net +3V3: track 0.00 -> 133.0 mm
- net N$3: track 0.00 -> 68.7 mm
- net PB0: track 0.00 -> 34.2 mm, vias 0 -> 1
- net PB1: track 0.00 -> 29.5 mm, vias 0 -> 1
- net PA14: track 0.00 -> 24.4 mm
- net PA13: track 0.00 -> 23.4 mm
- net PA7: track 0.00 -> 22.0 mm
- net PA6: track 0.00 -> 20.9 mm
- net PA15: track 0.00 -> 20.6 mm
- net PA5: track 0.00 -> 19.3 mm
- net PA0: track 0.00 -> 19.0 mm
- net PB3: track 0.00 -> 17.8 mm
- net PA1: track 0.00 -> 17.7 mm
- net +5V: track 0.00 -> 17.6 mm
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
Commit message: PCB003
Parts:
- moved LED1 106.8 mm to (58.4, 48.9), turned to 270 degrees
- moved R5 100.6 mm to (64.8, 44.5), turned to 270 degrees
- moved JP3 100.5 mm to (59.7, 37.5), turned to 90 degrees
- moved R4 92.4 mm to (61.6, 44.5), turned to 270 degrees
- moved LED3 88.3 mm to (64.8, 48.9), turned to 270 degrees
- moved R3 84.2 mm to (58.4, 44.5), turned to 270 degrees
- moved LED2 78.8 mm to (61.6, 48.9), turned to 270 degrees
- moved R2 52.2 mm to (31.1, 27.9), turned to 90 degrees
- moved C1 18.1 mm to (46.4, 17.1)
- moved C2 18.1 mm to (36.2, 17.1)
- moved JP4 18.1 mm to (55.2, 41.3)
- moved JP5 18.1 mm to (41.3, 52.7)
- moved Y1 18.1 mm to (41.3, 22.2)
- moved JP1 18.1 mm to (38.7, 59.1)
- moved U$1 18.1 mm to (41.3, 36.2)
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Routing:
- net GND: track 185.6 -> 224.7 mm
- net PA0: track 19.0 -> 36.9 mm
- net UART_TX: track 16.0 -> 27.9 mm
- net PB1: track 29.5 -> 39.3 mm
- net +3V3: track 133.0 -> 142.0 mm
- net UART_RX: track 15.0 -> 23.1 mm
- net PB0: track 34.2 -> 31.0 mm
- net PB6: track 15.1 -> 12.5 mm
- net N$5: track 0.00 -> 1.97 mm
- net N$4: track 0.00 -> 1.97 mm
- net PB7: track 16.2 -> 14.6 mm
- net BOOT0: track 11.7 -> 12.9 mm
- net PB5: track 16.2 -> 15.1 mm
- net PB3: track 17.8 -> 18.4 mm
Other:
- outline, holes or cut-outs redrawn
