File: STMBreadboard.sch (EAGLE design)
At the start: 16 parts, among them IC1 REG1117, Y1 8MHz

Commit message: 4
Parts:
- added LED1, LED2, LED3, LED4: (no value), led:LEDSML0805
- added R3, R4, R5, R6: 330, rcl:R-EU_R1206
Connections:
- new net N$4: LED1.A, R3.1
- new net N$5: LED2.A, R4.1
- new net N$6: LED3.A, R5.1
- new net N$7: LED4.A, R6.1
- net +3V3: now also R6.2
- net GND: now also LED1.C, LED2.C, LED3.C, LED4.C
- net PA0: now also R5.2
- net UART_RX: now also R3.2
- net UART_TX: now also R4.2
Changed lines of the file:
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@@
 <part name="R2" library="rcl" deviceset="R-EU_" device="R1206" value="10k"/>
 <part name="+3V5" library="supply1" deviceset="+3V3" device=""/>
+<part name="LED1" library="led" deviceset="LED" device="SML0805"/>
+<part name="LED2" library="led" deviceset="LED" device="SML0805"/>
+<part name="R3" library="rcl" deviceset="R-EU_" device="R1206" value="330"/>
+<part name="R4" library="rcl" deviceset="R-EU_" device="R1206" value="330"/>
+<part name="GND10" library="supply1" deviceset="GND" device=""/>
+<part name="GND11" library="supply1" deviceset="GND" device=""/>
+<part name="LED3" library="led" deviceset="LED" device="SML0805"/>
+<part name="R5" library="rcl" deviceset="R-EU_" device="R1206" value="330"/>
+<part name="GND12" library="supply1" deviceset="GND" device=""/>
+<part name="LED4" library="led" deviceset="LED" device="SML0805"/>
+<part name="R6" library="rcl" deviceset="R-EU_" device="R1206" value="330"/>
+<part name="GND13" library="supply1" deviceset="GND" device=""/>
 </parts>
 <sheets>
@@
 <instance part="R2" gate="G$1" x="-88.9" y="-27.94" rot="R90"/>
 <instance part="+3V5" gate="G$1" x="-88.9" y="0"/>
+<instance part="LED1" gate="G$1" x="71.12" y="68.58" rot="R90"/>
+<instance part="LED2" gate="G$1" x="71.12" y="81.28" rot="R90"/>
+<instance part="R3" gate="G$1" x="55.88" y="68.58" rot="R180"/>
+<instance part="R4" gate="G$1" x="55.88" y="81.28" rot="R180"/>
+<instance part="GND10" gate="1" x="81.28" y="76.2"/>
+<instance part="GND11" gate="1" x="81.28" y="63.5"/>
+<instance part="LED3" gate="G$1" x="71.12" y="55.88" rot="R90"/>
+<instance part="R5" gate="G$1" x="55.88" y="55.88" rot="R180"/>
+<instance part="GND12" gate="1" x="81.28" y="50.8"/>
+<instance part="LED4" gate="G$1" x="124.46" y="81.28" rot="R90"/>
+<instance part="R6" gate="G$1" x="109.22" y="81.28" rot="R180"/>
+<instance part="GND13" gate="1" x="134.62" y="76.2"/>
 </instances>
 <busses>
@@
 <pinref part="R2" gate="G$1" pin="1"/>
 <wire x1="-88.9" y1="-35.56" x2="-88.9" y2="-33.02" width="0.1524" layer="91"/>
+</segment>
+<segment>
+<pinref part="GND11" gate="1" pin="GND"/>
+<wire x1="81.28" y1="68.58" x2="81.28" y2="66.04" width="0.1524" layer="91"/>
+<pinref part="LED1" gate="G$1" pin="C"/>
+<wire x1="76.2" y1="68.58" x2="81.28" y2="68.58" width="0.1524" layer="91"/>
+</segment>
+<segment>
+<pinref part="LED2" gate="G$1" pin="C"/>
+<pinref part="GND10" gate="1" pin="GND"/>
+<wire x1="76.2" y1="81.28" x2="81.28" y2="81.28" width="0.1524" layer="91"/>
+<wire x1="81.28" y1="81.28" x2="81.28" y2="78.74" width="0.1524" layer="91"/>
+</segment>
+<segment>
+<pinref part="LED3" gate="G$1" pin="C"/>
+<pinref part="GND12" gate="1" pin="GND"/>
+<wire x1="76.2" y1="55.88" x2="81.28" y2="55.88" width="0.1524" layer="91"/>
+<wire x1="81.28" y1="55.88" x2="81.28" y2="53.34" width="0.1524" layer="91"/>
+</segment>
+<segment>
+<pinref part="LED4" gate="G$1" pin="C"/>
+<pinref part="GND13" gate="1" pin="GND"/>
+<wire x1="129.54" y1="81.28" x2="134.62" y2="81.28" width="0.1524" layer="91"/>
+<wire x1="134.62" y1="81.28" x2="134.62" y2="78.74" width="0.1524" layer="91"/>
 </segment>
 </net>
@@
 <wire x1="-88.9" y1="-15.24" x2="-88.9" y2="-2.54" width="0.1524" layer="91"/>
 </segment>
+<segment>
+<pinref part="R6" gate="G$1" pin="2"/>
+<wire x1="104.14" y1="81.28" x2="91.44" y2="81.28" width="0.1524" layer="91"/>
+<label x="91.44" y="81.28" size="1.778" layer="95"/>
+</segment>
 </net>
 <net name="PA14" class="0">
@@
 <pinref part="JP4" gate="A" pin="4"/>
 </segment>
+<segment>
+<pinref part="R3" gate="G$1" pin="2"/>
+<wire x1="50.8" y1="68.58" x2="38.1" y2="68.58" width="0.1524" layer="91"/>
+<label x="38.1" y="68.58" size="1.778" layer="95"/>
+</segment>
 </net>
 <net name="UART_TX" class="0">
@@
 <pinref part="JP4" gate="A" pin="3"/>
 </segment>
+<segment>
+<pinref part="R4" gate="G$1" pin="2"/>
+<wire x1="50.8" y1="81.28" x2="38.1" y2="81.28" width="0.1524" layer="91"/>
+<label x="38.1" y="81.28" size="1.778" layer="95"/>
+</segment>
 </net>
 <net name="PA0" class="0">
@@
 <wire x1="53.34" y1="40.64" x2="76.2" y2="40.64" width="0.1524" layer="91"/>
 <label x="58.42" y="40.64" size="1.778" layer="95"/>
+</segment>
+<segment>
+<pinref part="R5" gate="G$1" pin="2"/>
+<wire x1="50.8" y1="55.88" x2="38.1" y2="55.88" width="0.1524" layer="91"/>
+<label x="38.1" y="55.88" size="1.778" layer="95"/>
 </segment>
 </net>
@@
 </segment>
 </net>
+<net name="N$4" class="0">
+<segment>
+<pinref part="LED1" gate="G$1" pin="A"/>
+<pinref part="R3" gate="G$1" pin="1"/>
+<wire x1="68.58" y1="68.58" x2="60.96" y2="68.58" width="0.1524" layer="91"/>
+</segment>
+</net>
+<net name="N$5" class="0">
+<segment>
+<pinref part="R4" gate="G$1" pin="1"/>
+<pinref part="LED2" gate="G$1" pin="A"/>
+<wire x1="60.96" y1="81.28" x2="68.58" y2="81.28" width="0.1524" layer="91"/>
+</segment>
+</net>
+<net name="N$6" class="0">
+<segment>
+<pinref part="R5" gate="G$1" pin="1"/>
+<pinref part="LED3" gate="G$1" pin="A"/>
+<wire x1="60.96" y1="55.88" x2="68.58" y2="55.88" width="0.1524" layer="91"/>
+</segment>
+</net>
+<net name="N$7" class="0">
+<segment>
+<pinref part="R6" gate="G$1" pin="1"/>
+<pinref part="LED4" gate="G$1" pin="A"/>
+<wire x1="114.3" y1="81.28" x2="121.92" y2="81.28" width="0.1524" layer="91"/>
+</segment>
+</net>

Commit message: 4
Parts:
- added JP8: 3VOUT, pinhead:PINHD-1X2
Connections:
- net +3V3: now also JP8.2
- net GND: now also JP8.1
Changed lines of the file:
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@@
 <part name="R6" library="rcl" deviceset="R-EU_" device="R1206" value="330"/>
 <part name="GND13" library="supply1" deviceset="GND" device=""/>
+<part name="JP8" library="pinhead" deviceset="PINHD-1X2" device="" value="3VOUT"/>
+<part name="+3V6" library="supply1" deviceset="+3V3" device=""/>
+<part name="GND14" library="supply1" deviceset="GND" device=""/>
 </parts>
 <sheets>
@@
 <instance part="R6" gate="G$1" x="109.22" y="81.28" rot="R180"/>
 <instance part="GND13" gate="1" x="134.62" y="76.2"/>
+<instance part="JP8" gate="G$1" x="-68.58" y="86.36" rot="R180"/>
+<instance part="+3V6" gate="G$1" x="-55.88" y="93.98"/>
+<instance part="GND14" gate="1" x="-55.88" y="78.74"/>
 </instances>
 <busses>
@@
 <wire x1="129.54" y1="81.28" x2="134.62" y2="81.28" width="0.1524" layer="91"/>
 <wire x1="134.62" y1="81.28" x2="134.62" y2="78.74" width="0.1524" layer="91"/>
+</segment>
+<segment>
+<pinref part="JP8" gate="G$1" pin="1"/>
+<pinref part="GND14" gate="1" pin="GND"/>
+<wire x1="-66.04" y1="83.82" x2="-55.88" y2="83.82" width="0.1524" layer="91"/>
+<wire x1="-55.88" y1="83.82" x2="-55.88" y2="81.28" width="0.1524" layer="91"/>
 </segment>
 </net>
@@
 <label x="91.44" y="81.28" size="1.778" layer="95"/>
 </segment>
-</net>
+<segment>
+<pinref part="JP8" gate="G$1" pin="2"/>
+<pinref part="+3V6" gate="G$1" pin="+3V3"/>
+<wire x1="-66.04" y1="86.36" x2="-55.88" y2="86.36" width="0.1524" layer="91"/>
+<wire x1="-55.88" y1="86.36" x2="-55.88" y2="91.44" width="0.1524" layer="91"/>
+</segment>
+</net>

Commit message: PCB002
Parts:
- added C4, C5: 47u, rcl:CPOL-EUUD-6,3X7,7
Connections:
- net +3V3: now also C4.+
- net +5V: now also C5.+
- net GND: now also C4.-, C5.-
Changed lines of the file:
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@@
 <part name="+3V6" library="supply1" deviceset="+3V3" device=""/>
 <part name="GND14" library="supply1" deviceset="GND" device=""/>
+<part name="C4" library="rcl" deviceset="CPOL-EU" device="UD-6,3X7,7" value="47u"/>
+<part name="C5" library="rcl" deviceset="CPOL-EU" device="UD-6,3X7,7" value="47u"/>
+<part name="GND15" library="supply1" deviceset="GND" device=""/>
+<part name="GND16" library="supply1" deviceset="GND" device=""/>
 </parts>
 <sheets>
@@
 <instance part="GND5" gate="1" x="-45.72" y="-7.62"/>
 <instance part="IC1" gate="G$1" x="-20.32" y="83.82"/>
-<instance part="P+1" gate="1" x="-38.1" y="83.82" rot="R90"/>
-<instance part="+3V4" gate="G$1" x="-2.54" y="83.82" rot="R270"/>
+<instance part="P+1" gate="1" x="-48.26" y="83.82" rot="R90"/>
+<instance part="+3V4" gate="G$1" x="5.08" y="83.82" rot="R270"/>
 <instance part="GND6" gate="1" x="-20.32" y="66.04"/>
 <instance part="JP2" gate="G$1" x="-68.58" y="58.42" rot="R180"/>
@@
 <instance part="+3V6" gate="G$1" x="-55.88" y="93.98"/>
 <instance part="GND14" gate="1" x="-55.88" y="78.74"/>
+<instance part="C4" gate="G$1" x="-2.54" y="76.2"/>
+<instance part="C5" gate="G$1" x="-38.1" y="76.2"/>
+<instance part="GND15" gate="1" x="-38.1" y="66.04"/>
+<instance part="GND16" gate="1" x="-2.54" y="66.04"/>
 </instances>
 <busses>
@@
 <wire x1="-66.04" y1="83.82" x2="-55.88" y2="83.82" width="0.1524" layer="91"/>
 <wire x1="-55.88" y1="83.82" x2="-55.88" y2="81.28" width="0.1524" layer="91"/>
+</segment>
+<segment>
+<pinref part="GND15" gate="1" pin="GND"/>
+<pinref part="C5" gate="G$1" pin="-"/>
+<wire x1="-38.1" y1="68.58" x2="-38.1" y2="71.12" width="0.1524" layer="91"/>
+</segment>
+<segment>
+<pinref part="GND16" gate="1" pin="GND"/>
+<pinref part="C4" gate="G$1" pin="-"/>
+<wire x1="-2.54" y1="68.58" x2="-2.54" y2="71.12" width="0.1524" layer="91"/>
 </segment>
 </net>
@@
 <pinref part="IC1" gate="G$1" pin="VOUT"/>
 <pinref part="+3V4" gate="G$1" pin="+3V3"/>
-<wire x1="-7.62" y1="83.82" x2="-5.08" y2="83.82" width="0.1524" layer="91"/>
+<wire x1="-7.62" y1="83.82" x2="-2.54" y2="83.82" width="0.1524" layer="91"/>
+<pinref part="C4" gate="G$1" pin="+"/>
+<wire x1="-2.54" y1="83.82" x2="2.54" y2="83.82" width="0.1524" layer="91"/>
+<wire x1="-2.54" y1="78.74" x2="-2.54" y2="83.82" width="0.1524" layer="91"/>
+<junction x="-2.54" y="83.82"/>
 </segment>
 <segment>
@@
 <pinref part="P+1" gate="1" pin="+5V"/>
 <pinref part="IC1" gate="G$1" pin="VIN"/>
-<wire x1="-35.56" y1="83.82" x2="-33.02" y2="83.82" width="0.1524" layer="91"/>
-<wire x1="-35.56" y1="83.82" x2="-33.02" y2="83.82" width="0.1524" layer="91"/>
-</segment>
-<segment>
+<wire x1="-45.72" y1="83.82" x2="-38.1" y2="83.82" width="0.1524" layer="91"/>
+<pinref part="C5" gate="G$1" pin="+"/>
+<wire x1="-38.1" y1="83.82" x2="-33.02" y2="83.82" width="0.1524" layer="91"/>
+<wire x1="-38.1" y1="78.74" x2="-38.1" y2="83.82" width="0.1524" layer="91"/>
+<junction x="-38.1" y="83.82"/>
+</segment>
+<segment>

Commit message: LED 0603
Parts:
- LED1, LED2: device led:LEDSML0805 -> led:LEDCHIPLED_0603
- LED3, LED4: device led:LEDSML0805 -> led:LEDSML0603
Changed lines of the file:
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@@
 <setting verticaltext="up"/>
 </settings>
-<grid distance="0.1" unitdist="inch" unit="inch" style="lines" multiple="1" display="yes" altdistance="0.01" altunitdist="inch" altunit="inch"/>
+<grid distance="0.1" unitdist="inch" unit="inch" style="lines" multiple="1" display="no" altdistance="0.01" altunitdist="inch" altunit="inch"/>
 <layers>
-<layer number="1" name="Top" color="4" fill="1" visible="no" active="no"/>
-<layer number="16" name="Bottom" color="1" fill="1" visible="no" active="no"/>
-<layer number="17" name="Pads" color="2" fill="1" visible="no" active="no"/>
-<layer number="18" name="Vias" color="2" fill="1" visible="no" active="no"/>
-<layer number="19" name="Unrouted" color="6" fill="1" visible="no" active="no"/>
-<layer number="20" name="Dimension" color="15" fill="1" visible="no" active="no"/>
-<layer number="21" name="tPlace" color="7" fill="1" visible="no" active="no"/>
-<layer number="22" name="bPlace" color="7" fill="1" visible="no" active="no"/>
-<layer number="23" name="tOrigins" color="15" fill="1" visible="no" active="no"/>
-<layer number="24" name="bOrigins" color="15" fill="1" visible="no" active="no"/>
-<layer number="25" name="tNames" color="7" fill="1" visible="no" active="no"/>
-<layer number="26" name="bNames" color="7" fill="1" visible="no" active="no"/>
-<layer number="27" name="tValues" color="7" fill="1" visible="no" active="no"/>
-<layer number="28" name="bValues" color="7" fill="1" visible="no" active="no"/>
+<layer number="1" name="Top" color="4" fill="1" visible="yes" active="no"/>
+<layer number="16" name="Bottom" color="1" fill="1" visible="yes" active="no"/>
+<layer number="17" name="Pads" color="2" fill="1" visible="yes" active="no"/>
+<layer number="18" name="Vias" color="2" fill="1" visible="yes" active="no"/>
+<layer number="19" name="Unrouted" color="6" fill="1" visible="yes" active="no"/>
+<layer number="20" name="Dimension" color="15" fill="1" visible="yes" active="no"/>
+<layer number="21" name="tPlace" color="7" fill="1" visible="yes" active="no"/>
+<layer number="22" name="bPlace" color="7" fill="1" visible="yes" active="no"/>
+<layer number="23" name="tOrigins" color="15" fill="1" visible="yes" active="no"/>
+<layer number="24" name="bOrigins" color="15" fill="1" visible="yes" active="no"/>
+<layer number="25" name="tNames" color="7" fill="1" visible="yes" active="no"/>
+<layer number="26" name="bNames" color="7" fill="1" visible="yes" active="no"/>
+<layer number="27" name="tValues" color="7" fill="1" visible="yes" active="no"/>
+<layer number="28" name="bValues" color="7" fill="1" visible="yes" active="no"/>
 <layer number="29" name="tStop" color="7" fill="3" visible="no" active="no"/>
 <layer number="30" name="bStop" color="7" fill="6" visible="no" active="no"/>
@@
 <layer number="35" name="tGlue" color="7" fill="4" visible="no" active="no"/>
 <layer number="36" name="bGlue" color="7" fill="5" visible="no" active="no"/>
-<layer number="37" name="tTest" color="7" fill="1" visible="no" active="no"/>
-<layer number="38" name="bTest" color="7" fill="1" visible="no" active="no"/>
+<layer number="37" name="tTest" color="7" fill="1" visible="yes" active="no"/>
+<layer number="38" name="bTest" color="7" fill="1" visible="yes" active="no"/>
 <layer number="39" name="tKeepout" color="4" fill="11" visible="no" active="no"/>
 <layer number="40" name="bKeepout" color="1" fill="11" visible="no" active="no"/>
@@
 <layer number="44" name="Drills" color="7" fill="1" visible="no" active="no"/>
 <layer number="45" name="Holes" color="7" fill="1" visible="no" active="no"/>
-<layer number="46" name="Milling" color="3" fill="1" visible="no" active="no"/>
-<layer number="47" name="Measures" color="7" fill="1" visible="no" active="no"/>
-<layer number="48" name="Document" color="7" fill="1" visible="no" active="no"/>
-<layer number="49" name="Reference" color="7" fill="1" visible="no" active="no"/>
-<layer number="50" name="dxf" color="7" fill="1" visible="no" active="no"/>
-<layer number="51" name="tDocu" color="6" fill="1" visible="no" active="no"/>
-<layer number="52" name="bDocu" color="7" fill="1" visible="no" active="no"/>
-<layer number="53" name="tGND_GNDA" color="7" fill="9" visible="no" active="no"/>
-<layer number="54" name="bGND_GNDA" color="1" fill="9" visible="no" active="no"/>
-<layer number="56" name="wert" color="7" fill="1" visible="no" active="no"/>
-<layer number="57" name="tCAD" color="7" fill="1" visible="no" active="no"/>
+<layer number="46" name="Milling" color="3" fill="1" visible="yes" active="no"/>
+<layer number="47" name="Measures" color="7" fill="1" visible="yes" active="no"/>
+<layer number="48" name="Document" color="7" fill="1" visible="yes" active="no"/>
+<layer number="49" name="Reference" color="7" fill="1" visible="yes" active="no"/>
+<layer number="50" name="dxf" color="7" fill="1" visible="yes" active="no"/>
+<layer number="51" name="tDocu" color="7" fill="1" visible="yes" active="no"/>
+<layer number="52" name="bDocu" color="7" fill="1" visible="yes" active="no"/>
+<layer number="53" name="tGND_GNDA" color="7" fill="9" visible="yes" active="no"/>
+<layer number="54" name="bGND_GNDA" color="1" fill="9" visible="yes" active="no"/>
+<layer number="56" name="wert" color="7" fill="1" visible="yes" active="no"/>
+<layer number="57" name="tCAD" color="7" fill="1" visible="yes" active="no"/>
 <layer number="90" name="Modules" color="5" fill="1" visible="yes" active="yes"/>
 <layer number="91" name="Nets" color="2" fill="1" visible="yes" active="yes"/>
@@
 <part name="R2" library="rcl" deviceset="R-EU_" device="R1206" value="10k"/>
 <part name="+3V5" library="supply1" deviceset="+3V3" device=""/>
-<part name="LED1" library="led" deviceset="LED" device="SML0805"/>
-<part name="LED2" library="led" deviceset="LED" device="SML0805"/>
+<part name="LED1" library="led" deviceset="LED" device="CHIPLED_0603"/>
+<part name="LED2" library="led" deviceset="LED" device="CHIPLED_0603"/>
 <part name="R3" library="rcl" deviceset="R-EU_" device="R1206" value="330"/>
 <part name="R4" library="rcl" deviceset="R-EU_" device="R1206" value="330"/>
 <part name="GND10" library="supply1" deviceset="GND" device=""/>
 <part name="GND11" library="supply1" deviceset="GND" device=""/>
-<part name="LED3" library="led" deviceset="LED" device="SML0805"/>
+<part name="LED3" library="led" deviceset="LED" device="SML0603"/>
 <part name="R5" library="rcl" deviceset="R-EU_" device="R1206" value="330"/>
 <part name="GND12" library="supply1" deviceset="GND" device=""/>
-<part name="LED4" library="led" deviceset="LED" device="SML0805"/>
+<part name="LED4" library="led" deviceset="LED" device="SML0603"/>
 <part name="R6" library="rcl" deviceset="R-EU_" device="R1206" value="330"/>
 <part name="GND13" library="supply1" deviceset="GND" device=""/>
